File: ublox_NINA-W102/NINA-W102_minimal_breakout.kicad_pcb (KiCad board)
At the start: 2 copper layers, 47 x 20.7 mm, 19 parts, among them J1 Conn_01x15, J2 Conn_01x15, J3 6_PIN_SERIAL_TARGETLOCK, SW1 BOOT, SW2 RESET, U1 NINA-W102

Commit message: Corrected silk and added GDG logo
Parts:
- added G***: LOGO, lib:GDG-logo-mono-withouttext-h5.6, B.Cu at (119.6, 108.2)
- moved ? 42.0 mm to (119.0, 129.2)
- moved G*** 0.75 mm to (128.0, 107.6)
Other:
- board text added: "rac.su/ninab"
- board text added: "rev.0.5"
- board text removed: "rev.0.4"
- board text removed: "www.rac.su"
Changed lines of the file:
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@@
-(kicad_pcb (version 20170919) (host pcbnew "(2017-09-19 revision dddaa7e69)-makepkg")
+(kicad_pcb (version 4) (host pcbnew 4.0.7-e2-6376~60~ubuntu17.10.1)
   (general
+    (links 0)
+    (no_connects 0)
+    (area 104.064999 95.987799 151.205001 116.864201)
     (thickness 1.6)
     (drawings 69)
     (tracks 543)
     (zones 0)
-    (modules 19)
+    (modules 20)
     (nets 34)
   )
@@
   (title_block
     (title "ublox NINA-W102 minimal breakout")
-    (date 2018-04-22)
-    (rev 0.4)
+    (date 2018-05-21)
+    (rev 0.5)
     (company "GDG Zürich")
     (comment 1 "Michel Racic")
@@
     (0 F.Cu signal hide)
     (31 B.Cu signal hide)
-    (32 B.Adhes user)
-    (33 F.Adhes user)
-    (34 B.Paste user)
-    (35 F.Paste user)
-    (36 B.SilkS user)
+    (32 B.Adhes user hide)
+    (33 F.Adhes user hide)
+    (34 B.Paste user hide)
+    (35 F.Paste user hide)
+    (36 B.SilkS user hide)
     (37 F.SilkS user)
-    (38 B.Mask user)
-    (39 F.Mask user)
-    (40 Dwgs.User user)
-    (41 Cmts.User user)
-    (42 Eco1.User user)
-    (43 Eco2.User user)
-    (44 Edge.Cuts user)
-    (45 Margin user)
-    (46 B.CrtYd user)
-    (47 F.CrtYd user)
-    (48 B.Fab user)
-    (49 F.Fab user)
+    (38 B.Mask user hide)
+    (39 F.Mask user hide)
+    (40 Dwgs.User user hide)
+    (41 Cmts.User user hide)
+    (42 Eco1.User user hide)
+    (43 Eco2.User user hide)
+    (44 Edge.Cuts user hide)
+    (45 Margin user hide)
+    (46 B.CrtYd user hide)
+    (47 F.CrtYd user hide)
+    (48 B.Fab user hide)
+    (49 F.Fab user hide)
   )
   (setup
@@
       (usegerberextensions false)
       (usegerberattributes true)
-      (usegerberadvancedattributes true)
-      (creategerberjobfile true)
       (excludeedgelayer true)
       (linewidth 0.100000)
@@
       (hpglpenspeed 20)
       (hpglpendiameter 15)
+      (hpglpenoverlay 2)
       (psnegative false)
       (psa4output false)
@@
   )
   (module lib:DuckTapeApproved-MIT (layer B.Cu)
-    (at 127.254 107.696 180)
+    (at 128 107.6 180)
     (fp_text reference G*** (at 0 0 180) (layer B.SilkS) hide
       (effects (font (thickness 0.3)) (justify mirror))
@@
     (fp_line (start 7.62 1.524) (end -7.62 1.524) (layer F.SilkS) (width 0.127))
     (fp_line (start -7.62 1.524) (end -7.62 -1.27) (layer F.SilkS) (width 0.127))
-    (fp_text user GRN (at -8.509 -0.254) (layer F.SilkS)
+    (fp_text user GRN (at -8.509 -0.254 360) (layer F.SilkS)
       (effects (font (size 1.27 1.27) (thickness 0.2032)))
     )
-    (fp_text user BLK (at 8.636 0) (layer F.SilkS)
+    (fp_text user BLK (at 8.636 0 360) (layer F.SilkS)
       (effects (font (size 1.27 1.27) (thickness 0.2032)))
     )
@@
   )
   (module lib:BREADBOARD_SPACING_80mm (layer F.Cu)
-    (at 83.7184 106.3498 90)
+    (at 119 129.2 90)
     (descr "BREADBOARD SPACING")
     (tags "BREADBOARD SPACING")
@@
     (tags "PLATED THROUGH HOLE -15 PIN LOCKING FOOTPRINT")
     (attr virtual)
-    (fp_text reference J1 (at -1.9558 -0.889 180) (layer F.SilkS)
+    (fp_text reference J1 (at -1.89 0.884 180) (layer F.SilkS)
       (effects (font (size 0.6096 0.6096) (thickness 0.127)))
     )
@@
       (net 1 +3V3) (solder_mask_margin 0.1016))
   )
-  (gr_text www.rac.su (at 114.7572 112.8014) (layer B.SilkS)
+  (module lib:GDG-logo-mono-withouttext-h5.6 (layer B.Cu)
+    (at 119.6 108.2 180)
+    (fp_text reference G*** (at 0 0 180) (layer B.SilkS) hide
+      (effects (font (thickness 0.3)) (justify mirror))
+    )
+    (fp_text value LOGO (at 0.75 0 180) (layer B.SilkS) hide
+      (effects (font (thickness 0.3)) (justify mirror))
+    )
+    (fp_poly (pts (xy 0.002349 -0.625808) (xy 0.084957 -0.758082) (xy 0.153369 -0.872866) (xy 0.200999 -0.958727)
+      (xy 0.221264 -1.004231) (xy 0.221544 -1.006429) (xy 0.205254 -1.041581) (xy 0.158726 -1.123529)
+      (xy 0.086003 -1.245618) (xy -0.008872 -1.40119) (xy -0.121857 -1.583591) (xy -0.248908 -1.786165)
+      (xy -0.328101 -1.911304) (xy -0.878452 -2.778125) (xy -1.344101 -2.786911) (xy -1.507839 -2.788954)
+      (xy -1.646377 -2.78869) (xy -1.748622 -2.786295) (xy -1.80348 -2.78195) (xy -1.80975 -2.779403)
+      (xy -1.793314 -2.750642) (xy -1.746788 -2.674979) (xy -1.674345 -2.558977) (xy -1.580162 -2.409197)
+      (xy -1.468411 -2.2322) (xy -1.343266 -2.034548) (xy -1.208903 -1.822801) (xy -1.069495 -1.603521)
+      (xy -0.929217 -1.38327) (xy -0.792242 -1.168609) (xy -0.662746 -0.966099) (xy -0.544901 -0.782301)
+      (xy -0.442883 -0.623778) (xy -0.360866 -0.497089) (xy -0.303024 -0.408797) (xy -0.278077 -0.371808)
+      (xy -0.216141 -0.283242) (xy 0.002349 -0.625808)) (layer B.SilkS) (width 0.01))
+    (fp_poly (pts (xy 0.390778 -1.2638) (xy 0.443077 -1.327852) (xy 0.518103 -1.436664) (xy 0.581781 -1.534634)
+      (xy 0.662885 -1.663372) (xy 0.729481 -1.773388) (xy 0.774948 -1.853434) (xy 0.792668 -1.892262)
+      (xy 0.792704 -1.893031) (xy 0.776467 -1.928308) (xy 0.732313 -2.00761) (xy 0.665953 -2.121102)
+      (xy 0.583099 -2.258945) (xy 0.52769 -2.3495) (xy 0.263721 -2.778125) (xy -0.188061 -2.786949)
+      (xy -0.370309 -2.78943) (xy -0.496769 -2.788191) (xy -0.575073 -2.782665) (xy -0.612857 -2.772288)
+      (xy -0.617753 -2.756495) (xy -0.617076 -2.755199) (xy -0.583216 -2.698029) (xy -0.523112 -2.599741)
+      (xy -0.442168 -2.468925) (xy -0.345788 -2.314175) (xy -0.239378 -2.144082) (xy -0.128343 -1.967239)
+      (xy -0.018086 -1.792238) (xy 0.085988 -1.627672) (xy 0.178473 -1.482131) (xy 0.253966 -1.364209)
+      (xy 0.307061 -1.282498) (xy 0.332354 -1.24559) (xy 0.332879 -1.244977) (xy 0.355835 -1.238258)
+      (xy 0.390778 -1.2638)) (layer B.SilkS) (width 0.01))
+    (fp_poly (pts (xy -1.317512 2.755179) (xy -0.851156 2.746375) (xy 0.256712 0.92075) (xy 0.444772 0.610278)
+      (xy 0.622791 0.315271) (xy 0.788065 0.040281) (xy 0.937889 -0.210139) (xy 1.069559 -0.431436)
+      (xy 1.18037 -0.619058) (xy 1.26762 -0.768452) (xy 1.328603 -0.875066) (xy 1.360615 -0.934347)
+      (xy 1.364914 -0.944901) (xy 1.34928 -0.98546) (xy 1.307498 -1.065853) (xy 1.24765 -1.172435)
+      (xy 1.177822 -1.291556) (xy 1.106098 -1.409571) (xy 1.04056 -1.512832) (xy 0.989294 -1.58769)
+      (xy 0.969441 -1.612546) (xy 0.95601 -1.609894) (xy 0.929506 -1.583695) (xy 0.888093 -1.531113)
+      (xy 0.829939 -1.449315) (xy 0.753208 -1.335465) (xy 0.656069 -1.18673) (xy 0.536686 -1.000275)
+      (xy 0.393226 -0.773266) (xy 0.223855 -0.502868) (xy 0.02674 -0.186247) (xy -0.199954 0.179432)
+      (xy -0.415118 0.527463) (xy -0.624277 0.866234) (xy -0.823757 1.189568) (xy -1.011041 1.493371)
+      (xy -1.183614 1.773553) (xy -1.338961 2.026021) (xy -1.474566 2.246684) (xy -1.587914 2.43145)
+      (xy -1.676488 2.576227) (xy -1.737774 2.676923) (xy -1.769256 2.729446) (xy -1.772997 2.736187)
+      (xy -1.747076 2.745426) (xy -1.668268 2.752144) (xy -1.547149 2.755901) (xy -1.3943 2.756255)
+      (xy -1.317512 2.755179)) (layer B.SilkS) (width 0.01))
+    (fp_poly (pts (xy -0.166688 2.760853) (xy 0.269875 2.759456) (xy 1.04775 1.482916) (xy 1.825625 0.206375)
+      (xy 1.825257 -0.015875) (xy 1.822567 -0.130098) (xy 1.81018 -0.216023) (xy 1.780947 -0.296245)
+      (xy 1.727718 -0.393354) (xy 1.682382 -0.467365) (xy 1.61514 -0.571561) (xy 1.559028 -0.651237)
+      (xy 1.523131 -0.693763) (xy 1.516794 -0.697552) (xy 1.484435 -0.674548) (xy 1.447841 -0.627062)
+      (xy 1.410503 -0.56751) (xy 1.345937 -0.462948) (xy 1.257566 -0.319009) (xy 1.148814 -0.141323)
+      (xy 1.023103 0.064479) (xy 0.883855 0.292765) (xy 0.734494 0.537903) (xy 0.578442 0.794263)
+      (xy 0.419122 1.056213) (xy 0.259957 1.318122) (xy 0.10437 1.574358) (xy -0.044218 1.81929)
+      (xy -0.182382 2.047287) (xy -0.306701 2.252717) (xy -0.413751 2.42995) (xy -0.500109 2.573353)
+      (xy -0.562354 2.677296) (xy -0.597062 2.736147) (xy -0.60325 2.747516) (xy -0.573413 2.752761)
+      (xy -0.491541 2.756976) (xy -0.369097 2.759811) (xy -0.217545 2.760916) (xy -0.166688 2.760853)) (layer B.SilkS) (width 0.01))
+  )
+  (gr_text rac.su/ninab (at 115.2 112.8) (layer B.SilkS)
     (effects (font (size 1.5 1.5) (thickness 0.3)) (justify mirror))
   )
@@
     (effects (font (size 0.5 0.5) (thickness 0.12)) (justify right))
   )
-  (gr_text rev.0.4 (at 123.2916 106.7816 90) (layer F.SilkS)
+  (gr_text rev.0.5 (at 123.2916 106.7816 90) (layer F.SilkS)
     (effects (font (size 0.8 0.8) (thickness 0.127)))
   )

Commit message: Fixed breadboard spacing helper component position
Parts:
- moved ? 32.7 mm to (95.6, 106.4)
Changed lines of the file:
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@@
 (kicad_pcb (version 4) (host pcbnew 4.0.7-e2-6376~60~ubuntu17.10.1)
   (general
-    (links 0)
+    (links 73)
     (no_connects 0)
     (area 104.064999 95.987799 151.205001 116.864201)
@@
     (0 F.Cu signal hide)
     (31 B.Cu signal hide)
-    (32 B.Adhes user hide)
-    (33 F.Adhes user hide)
-    (34 B.Paste user hide)
-    (35 F.Paste user hide)
+    (32 B.Adhes user)
+    (33 F.Adhes user)
+    (34 B.Paste user)
+    (35 F.Paste user)
     (36 B.SilkS user hide)
     (37 F.SilkS user)
-    (38 B.Mask user hide)
-    (39 F.Mask user hide)
-    (40 Dwgs.User user hide)
-    (41 Cmts.User user hide)
-    (42 Eco1.User user hide)
-    (43 Eco2.User user hide)
-    (44 Edge.Cuts user hide)
-    (45 Margin user hide)
-    (46 B.CrtYd user hide)
-    (47 F.CrtYd user hide)
-    (48 B.Fab user hide)
-    (49 F.Fab user hide)
+    (38 B.Mask user)
+    (39 F.Mask user)
+    (40 Dwgs.User user)
+    (41 Cmts.User user)
+    (42 Eco1.User user)
+    (43 Eco2.User user)
+    (44 Edge.Cuts user)
+    (45 Margin user)
+    (46 B.CrtYd user)
+    (47 F.CrtYd user)
+    (48 B.Fab user)
+    (49 F.Fab user)
   )
   (setup
@@
     (pad_to_mask_clearance 0.0508)
     (aux_axis_origin 0 0)
-    (visible_elements 7FFFFFFF)
+    (visible_elements 7FFDFFFF)
     (pcbplotparams
       (layerselection 0x00030_80000001)
@@
   )
   (module lib:BREADBOARD_SPACING_80mm (layer F.Cu)
-    (at 119 129.2 90)
+    (at 95.6 106.4 90)
     (descr "BREADBOARD SPACING")
     (tags "BREADBOARD SPACING")
