File: ublox_NINA-W102/NINA-W102_minimal_breakout.sch (KiCad schematic (older format))
At the start: 15 parts, among them J1 Conn_01x15, J2 Conn_01x15, J3 6_PIN_SERIAL_TARGETLOCK, SW1 BOOT, SW2 RESET, U1 NINA-W102

Commit message: Added footprints to local library and reassigned in schematic
Parts:
- J1, J2: footprint Connectors-SparkFun:1X15_LOCK -> lib:1X15_LOCK
- JP1: footprint Jumpers:SMT-JUMPER_2_NC_TRACE_SILK -> lib:SMT-JUMPER_2_NC_TRACE_SILK
Changed lines of the file:
@@
 F 0 "J2" H 9750 4150 50  0000 C CNN
 F 1 "Conn_01x15" H 9750 2550 50  0000 C CNN
-F 2 "Connectors-SparkFun:1X15_LOCK" H 9750 3350 50  0001 C CNN
+F 2 "lib:1X15_LOCK" H 9750 3350 50  0001 C CNN
 F 3 "" H 9750 3350 50  0001 C CNN
 	1    9750 3350
@@
 F 0 "J1" H 2200 4150 50  0000 C CNN
 F 1 "Conn_01x15" H 2200 2550 50  0000 C CNN
-F 2 "Connectors-SparkFun:1X15_LOCK" H 2200 3350 50  0001 C CNN
+F 2 "lib:1X15_LOCK" H 2200 3350 50  0001 C CNN
 F 3 "" H 2200 3350 50  0001 C CNN
 	1    2200 3350
@@
 F 0 "JP1" H 3600 4250 45  0000 L BNN
 F 1 "JUMPER-SMT_2_NC" H 3300 4350 39  0000 L BNN
-F 2 "Jumpers:SMT-JUMPER_2_NC_TRACE_SILK" H 3700 4350 20  0001 C CNN
+F 2 "lib:SMT-JUMPER_2_NC_TRACE_SILK" H 3700 4350 20  0001 C CNN
 F 3 "" H 3700 4150 60  0001 C CNN
 F 4 "Nothing to assemble" H 3700 4150 60  0001 C CNN "Assembly"

Commit message: Changed schematics to current PCB revision and added all digikey partnumbers visible in the BOM html output
Parts:
- C1, C2: Digikey (none) -> 732-8086-1-ND
- C3, C4: Digikey (none) -> 732-7692-1-ND
- D1: value PWR RED -> PWR GREEN; Digikey (none) -> 732-5032-1-ND
- J1, J2: Digikey (none) -> WM50014-15-ND
- R1: Digikey (none) -> 541-1.0KECT-ND
- R2, R3: Digikey (none) -> 541-4201-1-ND
- SW1, SW2: Digikey (none) -> EG2663TR-ND
- U1: Digikey (none) -> 672-1070-1-ND
Other:
- note added: "Power lines only for ERC validation purposes"
Changed lines of the file:
@@
 Title "ublox NINA-W102 minimal breakout"
 Date "2018-04-18"
-Rev "0.4"
+Rev "0.5"
 Comp "GDG Zürich"
 Comment1 "Michel Racic"
@@
 F 1 "NINA-W102" H 6400 3450 60  0000 C CNN
 F 2 "lib:NINA-W102" H 5400 4800 60  0001 C CNN
-F 3 "https://www.u-blox.com/sites/default/files/NINA-W10_DataSheet_%28UBX-17065507%29.pdf" H 3800 -800 79  0000 C CNN
+F 3 "https://www.u-blox.com/sites/default/files/NINA-W10_DataSheet_%28UBX-17065507%29.pdf" H 5750 6100 79  0000 C CNN
+F 4 "672-1070-1-ND" H 6350 3400 60  0001 C CNN "Digikey"
 	1    6350 3400
 	1    0    0    -1
@@
 F 2 "Capacitors_SMD:C_1206_HandSoldering" H 4350 4250 50  0001 C CNN
 F 3 "" H 4350 4250 50  0001 C CNN
+F 4 "732-8086-1-ND" H 4350 4250 60  0001 C CNN "Digikey"
 	1    4350 4250
 	1    0    0    -1
@@
 L +3.3V #PWR01
 U 1 1 5ACA54B5
-P 1400 2150
-F 0 "#PWR01" H 1400 2000 50  0001 C CNN
-F 1 "+3.3V" H 1400 2290 50  0000 C CNN
-F 2 "" H 1400 2150 50  0001 C CNN
-F 3 "" H 1400 2150 50  0001 C CNN
-	1    1400 2150
+P -2500 800
+F 0 "#PWR01" H -2500 650 50  0001 C CNN
+F 1 "+3.3V" H -2500 940 50  0000 C CNN
+F 2 "" H -2500 800 50  0001 C CNN
+F 3 "" H -2500 800 50  0001 C CNN
+	1    -2500 800
 	1    0    0    -1
 $EndComp
@@
 F 2 "Capacitors_SMD:C_1206_HandSoldering" H 4750 4250 50  0001 C CNN
 F 3 "" H 4750 4250 50  0001 C CNN
+F 4 "732-8086-1-ND" H 4750 4250 60  0001 C CNN "Digikey"
 	1    4750 4250
 	1    0    0    -1
@@
 F 2 "lib:1X15_LOCK" H 9750 3350 50  0001 C CNN
 F 3 "" H 9750 3350 50  0001 C CNN
+F 4 "WM50014-15-ND" H 9750 3350 60  0001 C CNN "Digikey"
 	1    9750 3350
 	1    0    0    -1
@@
 F 2 "lib:1X15_LOCK" H 2200 3350 50  0001 C CNN
 F 3 "" H 2200 3350 50  0001 C CNN
+F 4 "WM50014-15-ND" H 2200 3350 60  0001 C CNN "Digikey"
 	1    2200 3350
 	-1   0    0    -1
@@
 L PWR_FLAG #FLG02
 U 1 1 5AD50A1E
-P 1050 2300
-F 0 "#FLG02" H 1050 2375 50  0001 C CNN
-F 1 "PWR_FLAG" H 1050 2450 50  0000 C CNN
-F 2 "" H 1050 2300 50  0001 C CNN
-F 3 "" H 1050 2300 50  0001 C CNN
-	1    1050 2300
+P -2850 950
+F 0 "#FLG02" H -2850 1025 50  0001 C CNN
+F 1 "PWR_FLAG" H -2850 1100 50  0000 C CNN
+F 2 "" H -2850 950 50  0001 C CNN
+F 3 "" H -2850 950 50  0001 C CNN
+	1    -2850 950
 	1    0    0    -1
 $EndComp
@@
 F 2 "switchessilicone:TACTILE_SWITCH_SMD_6.0X6.0MM" H 10300 4400 50  0001 C CNN
 F 3 "" H 10300 4400 50  0001 C CNN
+F 4 "EG2663TR-ND" H 10300 4200 60  0001 C CNN "Digikey"
 	1    10300 4200
 	0    1    1    0
@@
 F 2 "Capacitors_SMD:C_1206_HandSoldering" H 10600 4200 50  0001 C CNN
 F 3 "" H 10600 4200 50  0001 C CNN
+F 4 "732-7692-1-ND" H 10600 4200 60  0001 C CNN "Digikey"
 	1    10600 4200
 	1    0    0    -1
@@
 F 2 "Resistors_SMD:R_1206_HandSoldering" V 10380 3500 50  0001 C CNN
 F 3 "" H 10450 3500 50  0001 C CNN
+F 4 "541-4201-1-ND" V 10450 3500 60  0001 C CNN "Digikey"
 	1    10450 3500
 	1    0    0    -1
@@
 F 2 "switchessilicone:TACTILE_SWITCH_SMD_6.0X6.0MM" H 10300 2350 50  0001 C CNN
 F 3 "" H 10300 2350 50  0001 C CNN
+F 4 "EG2663TR-ND" H 10300 2150 60  0001 C CNN "Digikey"
 	1    10300 2150
 	0    1    1    0
@@
 F 2 "Capacitors_SMD:C_1206_HandSoldering" H 10600 2150 50  0001 C CNN
 F 3 "" H 10600 2150 50  0001 C CNN
+F 4 "732-7692-1-ND" H 10600 2150 60  0001 C CNN "Digikey"
 	1    10600 2150
 	1    0    0    -1
@@
 F 2 "Resistors_SMD:R_1206_HandSoldering" V 10380 1450 50  0001 C CNN
 F 3 "" H 10450 1450 50  0001 C CNN
+F 4 "541-4201-1-ND" V 10450 1450 60  0001 C CNN "Digikey"
 	1    10450 1450
 	1    0    0    -1
@@
 P 2950 4200
 F 0 "D1" H 2900 4325 50  0000 L CNN
-F 1 "PWR RED" H 2700 4100 50  0000 L CNN
+F 1 "PWR GREEN" H 2600 4100 50  0000 L CNN
 F 2 "LEDs:LED_1206_HandSoldering" V 2950 4200 50  0001 C CNN
 F 3 "" V 2950 4200 50  0001 C CNN
+F 4 "732-5032-1-ND" H 2950 4200 60  0001 C CNN "Digikey"
 	1    2950 4200
 	0    -1   -1   0
@@
 F 2 "Resistors_SMD:R_1206_HandSoldering" V 2880 4450 50  0001 C CNN
 F 3 "" H 2950 4450 50  0001 C CNN
+F 4 "541-1.0KECT-ND" V 2950 4450 60  0001 C CNN "Digikey"
 	1    2950 4450
 	1    0    0    -1
@@
 Connection ~ 900  3650
 Wire Wire Line
-	1400 2150 1400 2650
-Connection ~ 1400 2300
+	-2500 800  -2500 1300
+Connection ~ -2500 950
 Connection ~ 6300 4650
 Wire Wire Line
@@
 VCC
 Wire Wire Line
-	1400 2300 1050 2300
-Text Label 1400 2650 0    60   ~ 0
+	-2500 950  -2850 950
+Text Label -2500 1300 0    60   ~ 0
 VCC
 Text Label 10450 1150 0    60   ~ 0
@@
 Wire Wire Line
 	9550 3550 8400 3550
-Text Label 1400 1500 0    60   ~ 0
+Text Label -1450 1300 0    60   ~ 0
 VCC_IO
 Wire Wire Line
-	1400 800  1400 1500
+	-1450 600  -1450 1300
 $Comp
 L +1V8 #PWR_IO05
 U 1 1 5AD5EE0C
-P 1400 800
-F 0 "#PWR_IO05" H 1400 650 50  0001 C CNN
-F 1 "+1V8" H 1400 940 50  0000 C CNN
-F 2 "" H 1400 800 50  0001 C CNN
-F 3 "" H 1400 800 50  0001 C CNN
-	1    1400 800
-	1    0    0    -1
-$EndComp
+P -1450 600
+F 0 "#PWR_IO05" H -1450 450 50  0001 C CNN
+F 1 "+1V8" H -1450 740 50  0000 C CNN
+F 2 "" H -1450 600 50  0001 C CNN
+F 3 "" H -1450 600 50  0001 C CNN
+	1    -1450 600
+	1    0    0    -1
+$EndComp
+Text Notes -3150 250  0    60   Italic 0
+Power lines only for ERC validation purposes
 $EndSCHEMATC

Commit message: save
Parts:
- J3: Field4 Serial -> (none)
Changed lines of the file:
@@
 F 2 "lib:6_PIN_SERIAL_TARGET_SIDE_W_SILK" H 3400 7400 20  0001 C CNN
 F 3 "" H 3400 6700 50  0001 C CNN
-F 4 "Serial" H 3400 7450 60  0000 C CNN "Field4"
-F 5 "Left unpopulated" H 3400 6700 60  0001 C CNN "Assembly"
+F 4 "Left unpopulated" H 3400 6700 60  0001 C CNN "Assembly"
 	1    3400 6700
 	1    0    0    -1

Commit message: Added manufacturing output and corrected I2C issue with the badge carrier board
Parts:
- C3: Assembly (none) -> Leave unpopulated
Changed lines of the file:
@@
 Sheet 1 1
 Title "ublox NINA-W102 minimal breakout"
-Date "2018-04-18"
-Rev "0.5"
+Date "2018-06-21"
+Rev "0.5.1"
 Comp "GDG Zürich"
 Comment1 "Michel Racic"
@@
 F 3 "" H 10600 2150 50  0001 C CNN
 F 4 "732-7692-1-ND" H 10600 2150 60  0001 C CNN "Digikey"
+F 5 "Leave unpopulated" H 10600 2150 60  0001 C CNN "Assembly"
 	1    10600 2150
 	1    0    0    -1
